File: H-field_RF_probe.kicad_pcb (KiCad board)
At the start: 4 copper layers, 100 x 100 mm, 14 parts

Commit message: updated to v2.0 files
Parts:
- removed ? (x6): MountingHole_3.2mm_M3_Pad_Via_noFmask, User:MountingHole_3.2mm_M3_Pad_Via_noFmask
- removed ? (x4): Fiducial_0.5mm_Dia_1mm_Outer, Fiducials:Fiducial_0.5mm_Dia_1mm_Outer
- removed svg2mod: G***, User:MR_Engineering_logo_14mm_text
- added G***: LOGO, Logo:MR_Engineering_logo_12mm, F.Cu at (161.0, 65.0)
- added REF**: MountingHole_3.2mm_M3, MountingHole:MountingHole_3.2mm_M3, F.Cu at (142.0, 58.0)
- added REF**: MountingHole_3.2mm_M3, MountingHole:MountingHole_3.2mm_M3, F.Cu at (108.0, 58.0)
- added REF**: MountingHole_3.2mm_M3, MountingHole:MountingHole_3.2mm_M3, F.Cu at (175.0, 73.0)
- added REF**: MountingHole_3.2mm_M3, MountingHole:MountingHole_3.2mm_M3, F.Cu at (175.0, 58.0)
- added REF**: MountingHole_3.2mm_M3, MountingHole:MountingHole_3.2mm_M3, F.Cu at (142.0, 73.0)
- added REF**: MountingHole_3.2mm_M3, MountingHole:MountingHole_3.2mm_M3, F.Cu at (108.0, 73.0)
- moved REF*** 8.02 mm to (112.0, 65.0)
- moved G*** 6.26 mm to (130.0, 65.0)
Routing:
- net /signal: track 131.2 -> 77.7 mm
- net GND: vias 285 -> 185
- net (no net): vias 4 -> 0
- added copper zone on In1.Cu, net GND
- added copper zone on In2.Cu, net GND
- removed copper zone on Signal.Cu, net GND
- removed copper zone on middle.Cu, net GND
Other:
- board size 100 x 100 mm -> 99.5 x 23 mm
- net class Default removed
- board text added: "Rev. 1.1 2023-05-15"
- board text added: "https://github.com/dezanche CERN OHL-W v2"
- board text removed: "V cut →"
- board text removed: "https://github.com/dezanche CERN OHL v1.2 Rev. 1, 2019-04-05"
